Commit message: modified:   Dockerfile 	modified:   ros2_ws/commands.txt 	modified:   ros2_ws/src/goosebot_0/CMakeLists.txt 	modified:   ros2_ws/src/goosebot_0/config/nav2_params.yaml 	modified:   ros2_ws/src/goosebot_0/launch/nav2_bringup.launch.py 	modified:   ros2_ws/src/goosebot_0/launch/spawn_robot.launch.py 	modified:   ros2_ws/src/goosebot_0/package.xml 	modified:   ros2_ws/src/goosebot_0/urdf/robot.urdf.xacro 	ros2_ws/src/goosebot_0/maps/ 	ros2_ws/src/goosebot_0/scripts/

File: 11_sim_nav2/ros2_ws/src/goosebot_0/urdf/robot.urdf.xacro (robot description, xacro)
@@ -138,5 +138,5 @@
   <!-- edge height. Update x/y/z below once that's decided.          -->
   <!-- ============================================================ -->
-  <xacro:property name="tof_x_offset" value="${base_length/2}"/>
+  <xacro:property name="tof_x_offset" value="${base_length/2 + 0.02}"/>
   <xacro:property name="tof_z_offset" value="0.0"/>
   <link name="tof_front_link">
@@ -210,7 +210,8 @@
   <gazebo reference="tof_front_link">
     <sensor type="ray" name="tof_front_sensor">
-      <update_rate>20.0</update_rate>
-      <always_on>true</always_on>
-      <ray>
+	  <update_rate>20.0</update_rate>
+	  <always_on>true</always_on>
+	  <visualize>true</visualize>
+	  <ray>
         <scan>
           <horizontal>
@@ -221,13 +222,13 @@
           </horizontal>
           <vertical>
-            <samples>5</samples>
+            <samples>3</samples>
             <resolution>1</resolution>
-            <min_angle>-0.235</min_angle>
-            <max_angle>0.235</max_angle>
+            <min_angle>0.01</min_angle>
+            <max_angle>0.15</max_angle>
           </vertical>
         </scan>
         <range>
           <min>0.04</min>
-          <max>4.0</max>
+          <max>8.0</max>
           <resolution>0.001</resolution>
         </range>
@@ -248,4 +249,19 @@
       </plugin>
     </sensor>
+  </gazebo>
+  <!-- ============================================================ -->
+  <!-- GAZEBO GROUND TRUTH POSE - sim-only, feeds the perfect-map    -->
+  <!-- localization bridge. Not present on real hardware.            -->
+  <!-- ============================================================ -->
+  <gazebo>
+    <plugin name="ground_truth_p3d" filename="libgazebo_ros_p3d.so">
+      <ros>
+        <namespace>/ground_truth</namespace>
+        <remapping>odom:=pose</remapping>
+      </ros>
+      <body_name>base_footprint</body_name>
+      <frame_name>map</frame_name>
+      <update_rate>30.0</update_rate>
+    </plugin>
   </gazebo>
   <gazebo reference="imu_link">

Commit message: Removed old files and added EKF control

File: 11_sim_nav2/ros2_ws/src/goosebot_0/urdf/robot.urdf.xacro (robot description, xacro)
@@ -18,4 +18,7 @@
   <xacro:property name="camera_mount_height" value="0.09"/>
   <xacro:property name="camera_x_offset" value="0.05"/>
+  <!-- GPS antenna sits top-center, clear sky view. Placeholder height,
+       adjust once the hardware team picks a final enclosure/mast. -->
+  <xacro:property name="gps_z_offset" value="${base_height/2 + 0.02}"/>
   <!-- ============================================================ -->
   <!-- MATERIALS                                                     -->
@@ -156,16 +159,37 @@
   </joint>
   <!-- ============================================================ -->
+  <!-- GPS - top-center mount, placeholder position                 -->
+  <!-- Mount position is a placeholder like the ToF: hardware team   -->
+  <!-- hasn't picked final enclosure placement yet. Sensor/plugin    -->
+  <!-- block comes in a later step; this just establishes the        -->
+  <!-- frame so TF is correct first.                                 -->
+  <!-- ============================================================ -->
+  <link name="gps_link">
+    <visual>
+      <geometry><box size="0.02 0.02 0.01"/></geometry>
+      <material name="sensor_black"/>
+    </visual>
+    <inertial>
+      <mass value="0.01"/>
+      <inertia ixx="0.000001" ixy="0" ixz="0" iyy="0.000001" iyz="0" izz="0.000001"/>
+    </inertial>
+  </link>
+  <joint name="gps_joint" type="fixed">
+    <parent link="base_link"/>
+    <child link="gps_link"/>
+    <origin xyz="0 0 ${gps_z_offset}" rpy="0 0 0"/>
+  </joint>
+  <!-- ============================================================ -->
   <!-- GZ-SIM: skid-steer drive (4 independently driven wheels,      -->
   <!-- differential steering left-pair vs right-pair)                -->
   <!--                                                                -->
-  <!-- libgazebo_ros_diff_drive.so -> gz-sim-diff-drive-system.       -->
-  <!-- Same left/right joint pairs still work (DiffDrive supports     -->
-  <!-- multiple <left_joint>/<right_joint> entries for skid-steer).   -->
-  <!-- Two real changes: (1) it takes <wheel_radius>, not              -->
-  <!-- <wheel_diameter> — the old file's repeated wheel_diameter tag  -->
-  <!-- is now just wheel_radius once. (2) it no longer talks ROS       -->
-  <!-- directly: cmd_vel comes in and odom/tf go out over gz-transport -->
-  <!-- on the <topic>/<odom_topic>/<tf_topic> names below, which the   -->
-  <!-- ros_gz_bridge config bridges to /cmd_vel, /odom, and /tf.       -->
+  <!-- gz-sim 8's DiffDrive has NO publish_odom / publish_odom_tf /   -->
+  <!-- publish_wheel_tf switches (not in its documented parameter     -->
+  <!-- list); those tags were silently ignored and DiffDrive kept     -->
+  <!-- publishing its own odom->base_footprint TF. They are removed,  -->
+  <!-- and <frame_id>/<child_frame_id>/<tf_topic> are left at their   -->
+  <!-- namespaced defaults (<model>/odom, /model/<name>/tf) so this   -->
+  <!-- plugin can never collide with the EKF's odom->base_footprint.  -->
+  <!-- Real odom TF comes from robot_localization only.               -->
   <!-- ============================================================ -->
   <gazebo>
@@ -183,12 +207,5 @@
       <max_wheel_acceleration>2.0</max_wheel_acceleration>
       <topic>cmd_vel</topic>
-      <odom_topic>odom</odom_topic>
-      <tf_topic>tf</tf_topic>
-      <frame_id>odom</frame_id>
-      <child_frame_id>base_footprint</child_frame_id>
       <odom_publish_frequency>50</odom_publish_frequency>
-      <publish_odom>true</publish_odom>
-      <publish_odom_tf>true</publish_odom_tf>
-      <publish_wheel_tf>true</publish_wheel_tf>
     </plugin>
   </gazebo>
@@ -209,4 +226,5 @@
       <update_rate>30.0</update_rate>
       <topic>camera/image</topic>
+      <gz_frame_id>camera_optical_link</gz_frame_id>
       <camera>
         <horizontal_fov>1.5708</horizontal_fov>
@@ -242,4 +260,5 @@
       <visualize>true</visualize>
       <topic>tof_front/scan</topic>
+      <gz_frame_id>tof_front_link</gz_frame_id>
       <lidar>
         <scan>
@@ -271,4 +290,43 @@
   </gazebo>
   <!-- ============================================================ -->
+  <!-- GZ-SIM: GPS (NavSat) sensor                                    -->
+  <!--                                                                -->
+  <!-- Like the camera/IMU, this is native to Harmonic's Sensors      -->
+  <!-- system; no separate plugin needed, just a <sensor              -->
+  <!-- type="navsat"> block. It emits gz.msgs.NavSat, which the       -->
+  <!-- bridge config (next step) maps to sensor_msgs/NavSatFix.       -->
+  <!--                                                                -->
+  <!-- update_rate is deliberately slow (5 Hz); real consumer GPS     -->
+  <!-- modules update at 1-10 Hz, much slower than IMU/ToF. Noise     -->
+  <!-- stddevs below are rough placeholders for an uncorrected        -->
+  <!-- consumer GPS (~1.5m horizontal, ~3m vertical); tighten these   -->
+  <!-- once you know the actual module (e.g. RTK would be far        -->
+  <!-- better than this).                                             -->
+  <!-- ============================================================ -->
+  <gazebo reference="gps_link">
+    <sensor type="navsat" name="gps_sensor">
+      <update_rate>5.0</update_rate>
+      <always_on>true</always_on>
+      <topic>gps/fix</topic>
+      <gz_frame_id>gps_link</gz_frame_id>
+      <navsat>
+        <position_sensing>
+          <horizontal>
+            <noise type="gaussian">
+              <mean>0.0</mean>
+              <stddev>1.5</stddev>
+            </noise>
+          </horizontal>
+          <vertical>
+            <noise type="gaussian">
+              <mean>0.0</mean>
+              <stddev>3.0</stddev>
+            </noise>
+          </vertical>
+        </position_sensing>
+      </navsat>
+    </sensor>
+  </gazebo>
+  <!-- ============================================================ -->
   <!-- GZ-SIM GROUND TRUTH POSE - sim-only, feeds the perfect-map    -->
   <!-- localization bridge. Not present on real hardware.             -->
@@ -305,4 +363,5 @@
       <update_rate>100.0</update_rate>
       <topic>imu/data</topic>
+      <gz_frame_id>imu_link</gz_frame_id>
       <imu>
         <angular_velocity>

Commit message: Fixed an EKF bug causing drifting rotation

File: 11_sim_nav2/ros2_ws/src/goosebot_0/urdf/robot.urdf.xacro (robot description, xacro)
@@ -18,4 +18,14 @@
   <xacro:property name="camera_mount_height" value="0.09"/>
   <xacro:property name="camera_x_offset" value="0.05"/>
+  <!-- STEREO RIG. Baseline defaults to the width of the existing camera_link
+       bar (0.09 m), PLACEHOLDER: set to your real rig's baseline. The
+       camera_info fixer node (scripts/stereo_camera_info_fixer.py) reads the
+       same number via the launch arg 'baseline'; keep the two in sync.
+       FOV/resolution carried over from the old single camera (provisional). -->
+  <xacro:property name="stereo_baseline" value="0.09"/>
+  <xacro:property name="stereo_hfov"     value="1.5708"/>
+  <xacro:property name="stereo_width"    value="640"/>
+  <xacro:property name="stereo_height"   value="480"/>
+  <xacro:property name="stereo_fps"      value="20.0"/>
   <!-- GPS antenna sits top-center, clear sky view. Placeholder height,
        adjust once the hardware team picks a final enclosure/mast. -->
@@ -114,11 +124,49 @@
     <origin xyz="0 0 ${camera_mount_height/2}" rpy="0 0 0"/>
   </joint>
-  <!-- optical frame, so image data uses the standard camera convention -->
-  <link name="camera_optical_link"/>
-  <joint name="camera_optical_joint" type="fixed">
-    <parent link="camera_link"/>
-    <child link="camera_optical_link"/>
-    <origin xyz="0 0 0" rpy="${-pi/2} 0 ${-pi/2}"/>
-  </joint>
+  <!-- ============================================================ -->
+  <!-- STEREO PAIR: camera_link is the rig's center; the two imagers   -->
+  <!-- sit at +/- stereo_baseline/2 along its Y axis (left = +Y, ROS   -->
+  <!-- convention). Each imager is an x-forward link (the direction a  -->
+  <!-- gz camera sensor looks) with a child *_optical_link carrying    -->
+  <!-- the z-forward optical convention; gz_frame_id points at the     -->
+  <!-- optical link so image/camera_info headers match TF.             -->
+  <!-- Both imagers are parallel and distortion-free, i.e. the images  -->
+  <!-- are already rectified, so no stereo_image_proc needed in sim.    -->
+  <!-- ============================================================ -->
+  <xacro:macro name="stereo_imager" params="side y_offset">
+    <link name="camera_${side}_link">
+      <inertial>
+        <mass value="0.01"/>
+        <inertia ixx="0.000001" ixy="0" ixz="0" iyy="0.000001" iyz="0" izz="0.000001"/>
+      </inertial>
+    </link>
+    <joint name="camera_${side}_joint" type="fixed">
+      <parent link="camera_link"/>
+      <child link="camera_${side}_link"/>
+      <origin xyz="0 ${y_offset} 0" rpy="0 0 0"/>
+    </joint>
+    <link name="camera_${side}_optical_link"/>
+    <joint name="camera_${side}_optical_joint" type="fixed">
+      <parent link="camera_${side}_link"/>
+      <child link="camera_${side}_optical_link"/>
+      <origin xyz="0 0 0" rpy="${-pi/2} 0 ${-pi/2}"/>
+    </joint>
+    <gazebo reference="camera_${side}_link">
+      <sensor type="camera" name="stereo_${side}">
+        <always_on>true</always_on>
+        <update_rate>${stereo_fps}</update_rate>
+        <topic>stereo/${side}/image</topic>
+        <gz_frame_id>camera_${side}_optical_link</gz_frame_id>
+        <camera>
+          <camera_info_topic>stereo/${side}/camera_info</camera_info_topic>
+          <horizontal_fov>${stereo_hfov}</horizontal_fov>
+          <image><width>${stereo_width}</width><height>${stereo_height}</height><format>R8G8B8</format></image>
+          <clip><near>0.02</near><far>300</far></clip>
+        </camera>
+      </sensor>
+    </gazebo>
+  </xacro:macro>
+  <xacro:stereo_imager side="left"  y_offset="${stereo_baseline/2}"/>
+  <xacro:stereo_imager side="right" y_offset="${-stereo_baseline/2}"/>
   <!-- ============================================================ -->
   <!-- IMU                                                           -->
@@ -209,31 +257,4 @@
       <odom_publish_frequency>50</odom_publish_frequency>
     </plugin>
-  </gazebo>
-  <!-- ============================================================ -->
-  <!-- GZ-SIM: camera sensor                                          -->
-  <!--                                                                -->
-  <!-- libgazebo_ros_camera.so is gone entirely — Harmonic's Sensors  -->
-  <!-- system (loaded once at the world level in maze.world) natively  -->
-  <!-- simulates any <sensor type="camera"> and auto-publishes it on   -->
-  <!-- gz-transport. The <topic> tag below just gives it a predictable -->
-  <!-- name instead of the generated default, so the bridge config can -->
-  <!-- target it. horizontal_fov is still the same provisional         -->
-  <!-- placeholder noted below — swap in the calibrated value once    -->
-  <!-- you've run camera_calibration.                                  -->
-  <!-- ============================================================ -->
-  <gazebo reference="camera_link">
-    <sensor type="camera" name="front_camera">
-      <update_rate>30.0</update_rate>
-      <topic>camera/image</topic>
-      <gz_frame_id>camera_optical_link</gz_frame_id>
-      <camera>
-        <horizontal_fov>1.5708</horizontal_fov>
-        <image><width>640</width><height>480</height><format>R8G8B8</format></image>
-        <clip><near>0.02</near><far>300</far></clip>
-      </camera>
-      <!-- gz-sim publishes camera_info automatically alongside the
-           image topic; confirm the exact name once running with
-           `gz topic -l`, it should be camera/camera_info. -->
-    </sensor>
   </gazebo>
   <!-- ============================================================ -->
